File: electrical/pcb/Rainworks_Electrical.kicad_pcb (KiCad board)
At the start: 2 copper layers, 111.4 x 40.9 mm, 19 parts, among them J1 472192001, P1 ESP8266 Thing, U1 MCP3008, U10 S1_SM, U11 S0_PH, U7 S4_FR, U8 S3_T, U9 S2_C

Commit message: changes for routing with sd
Parts:
- C2, C3: moved to B.Cu
- U1: footprint DIP16-2.54-19.2X7.62MM -> Package_SO:SOIC-16_3.9x9.9mm_P1.27mm
- moved C3 17.1 mm to (191.9, 93.8), turned to 90 degrees
- moved C2 13.9 mm to (189.9, 96.6), turned to 90 degrees
- moved U1 4.50 mm to (165.5, 101.8), turned to 90 degrees
- moved J1 3.89 mm to (189.8, 99.5), turned to 180 degrees
Routing:
- net GND: track 192.1 -> 0.00 mm
- net (no net): track 105.0 -> 0.00 mm
- net /3V3_VDD: track 33.1 -> 123.1 mm, vias 0 -> 2
- net /VIN_5V0_MCU: track 0.00 -> 85.9 mm
- net /SD_MISO_SPI: track 85.4 -> 117.8 mm, vias 1 -> 0
- net /SD_SCLK_SPI: track 123.2 -> 94.6 mm, vias 0 -> 1
- net /CH4_ADC: track 8.80 -> 32.0 mm, vias 0 -> 2
- net /CH3_ADC: track 0.00 -> 20.4 mm
- net /SD_CS_SPI: track 80.1 -> 66.1 mm, vias 1 -> 0
- net /CH1_ADC: track 4.59 -> 16.2 mm, vias 0 -> 1
- net Net-(P1-15): track 45.5 -> 35.6 mm, vias 0 -> 1
- net /CH0_ADC: track 11.8 -> 15.7 mm, vias 0 -> 1
- net /S4_FR_VOUT: track 0.00 -> 3.68 mm
- net /CH2_ADC: track 14.7 -> 11.7 mm
- net /SD_MOSI_SPI: track 76.1 -> 78.7 mm, vias 0 -> 1
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Other:
- outline, holes or cut-outs redrawn
