File: electrical/pcb/Rainworks_Electrical.kicad_pcb (KiCad board)
At the start: 2 copper layers, 111.4 x 40.9 mm, 19 parts, among them J1 472192001, P1 ESP8266 Thing, U1 MCP3008, U10 S1_SM, U11 S0_PH, U7 S4_FR, U8 S3_T, U9 S2_C

Commit message: add test points to PCB
Parts:
- added TP1: TURB, Connector_PinHeader_2.54mm:PinHeader_1x01_P2.54mm_Vertical, F.Cu at (190.4, 113.8)
- added TP10: GND, Connector_PinHeader_2.54mm:PinHeader_1x01_P2.54mm_Vertical, F.Cu at (203.1, 111.6)
- added TP2: FR, Connector_PinHeader_2.54mm:PinHeader_1x01_P2.54mm_Vertical, F.Cu at (190.4, 117.9)
- added TP3: GND, Connector_PinHeader_2.54mm:PinHeader_1x01_P2.54mm_Vertical, F.Cu at (195.9, 113.9)
- added TP4: GND, Connector_PinHeader_2.54mm:PinHeader_1x01_P2.54mm_Vertical, F.Cu at (195.9, 117.8)
- added TP5: SDVDD, Connector_PinHeader_2.54mm:PinHeader_1x01_P2.54mm_Vertical, F.Cu at (203.0, 90.9)
- added TP6: MOSI, Connector_PinHeader_2.54mm:PinHeader_1x01_P2.54mm_Vertical, F.Cu at (203.4, 103.0)
- added TP7: MISO, Connector_PinHeader_2.54mm:PinHeader_1x01_P2.54mm_Vertical, F.Cu at (203.0, 95.1)
- added TP8: SCLK, Connector_PinHeader_2.54mm:PinHeader_1x01_P2.54mm_Vertical, F.Cu at (203.2, 107.0)
- added TP9: CS, Connector_PinHeader_2.54mm:PinHeader_1x01_P2.54mm_Vertical, F.Cu at (203.2, 99.2)
- moved C2 0.35 mm to (190.8, 99.5)
Routing:
- net /SD_SCLK_SPI: track 75.9 -> 115.2 mm, vias 2 -> 1
- net /CH4_ADC: track 27.5 -> 52.6 mm
- net /SD_MISO_SPI: track 68.6 -> 86.9 mm, vias 0 -> 3
- net /SD_CS_SPI: track 65.5 -> 82.4 mm, vias 0 -> 1
- net /3V3_VDD: track 122.3 -> 139.0 mm
- net /SD_MOSI_SPI: track 105.9 -> 91.1 mm
- net /CH3_ADC: track 17.2 -> 26.5 mm, vias 0 -> 1
- net /VIN_5V0_MCU: track 85.4 -> 88.6 mm, vias 0 -> 1
- net /CH1_ADC: track 17.4 -> 15.9 mm
- net Net-(P1-15): track 36.1 -> 37.3 mm
- net GND: track 3.05 -> 2.49 mm
