File: electrical/pcb/Rainworks_Electrical.kicad_sch (KiCad schematic)
At the start: 19 parts, among them J1 472192001, P1 ESP8266 Thing, U1 MCP3008, U10 S1_SM, U11 S0_PH, U7 S4_FR, U8 S3_T, U9 S2_C

Commit message: add test points to PCB
Parts:
- added TP1: T_TP, Connector_PinHeader_2.54mm:PinHeader_1x01_P2.54mm_Vertical, symbol Connector:TestPoint
- added TP2: FRTP, Connector_PinHeader_2.54mm:PinHeader_1x01_P2.54mm_Vertical, symbol Connector:TestPoint
- added TP3, TP4: GND, Connector_PinHeader_2.54mm:PinHeader_1x01_P2.54mm_Vertical, symbol Connector:TestPoint
- added TP5: SDVDD_TP, Connector_PinHeader_2.54mm:PinHeader_1x01_P2.54mm_Vertical, symbol Connector:TestPoint
- added TP6: MOSI_TP, Connector_PinHeader_2.54mm:PinHeader_1x01_P2.54mm_Vertical, symbol Connector:TestPoint
- added TP7: MISO_TP, Connector_PinHeader_2.54mm:PinHeader_1x01_P2.54mm_Vertical, symbol Connector:TestPoint
- added TP8: SCLK_TP, Connector_PinHeader_2.54mm:PinHeader_1x01_P2.54mm_Vertical, symbol Connector:TestPoint
- added TP9: CS_TP, Connector_PinHeader_2.54mm:PinHeader_1x01_P2.54mm_Vertical, symbol Connector:TestPoint
Connections:
- net 3V3_VDD: now also TP5.1
- net CH3_ADC: now also TP1.1
- net CH4_ADC: now also TP2.1
- net GND: now also TP3.1, TP4.1
- net SD_CS_SPI: now also TP9.1
- net SD_MISO_SPI: now also TP7.1
- net SD_MOSI_SPI: now also TP6.1
- net SD_SCLK_SPI: now also TP8.1

Commit message: extra changes for tp
Parts:
- added TP10: GND, Connector_PinHeader_2.54mm:PinHeader_1x01_P2.54mm_Vertical, symbol Connector:TestPoint
Connections:
- net GND: now also TP10.1
Other:
- moved on the sheet: TP4
Changed lines of the file:
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@@
 	)
 	(junction
-		(at 121.92 185.42)
-		(diameter 0)
-		(color 0 0 0 0)
-	)
-	(junction
 		(at 179.07 53.34)
 		(diameter 0)
@@
 	)
 	(junction
+		(at 125.73 185.42)
+		(diameter 0)
+		(color 0 0 0 0)
+	)
+	(junction
 		(at 78.232 120.65)
 		(diameter 0)
@@
 	)
 	(junction
+		(at 116.84 185.42)
+		(diameter 0)
+		(color 0 0 0 0)
+	)
+	(junction
 		(at 119.126 53.34)
 		(diameter 0)
@@
 	(wire
 		(pts
-			(xy 105.41 185.42) (xy 121.92 185.42)
+			(xy 105.41 185.42) (xy 116.84 185.42)
 		)
 		(stroke
@@
 	(wire
 		(pts
-			(xy 121.92 185.42) (xy 135.89 185.42)
-		)
-		(stroke
-			(width 0)
-			(type default)
-		)
-	)
-	(wire
-		(pts
 			(xy 184.15 117.602) (xy 189.23 117.602)
 		)
@@
 	(wire
 		(pts
+			(xy 116.84 185.42) (xy 125.73 185.42)
+		)
+		(stroke
+			(width 0)
+			(type default)
+		)
+	)
+	(wire
+		(pts
 			(xy 119.126 53.34) (xy 119.126 105.664)
 		)
@@
 	(wire
 		(pts
+			(xy 125.73 185.42) (xy 135.89 185.42)
+		)
+		(stroke
+			(width 0)
+			(type default)
+		)
+	)
+	(wire
+		(pts
 			(xy 101.346 50.8) (xy 101.346 51.054)
 		)
@@
 	(symbol
 		(lib_id "Connector:TestPoint")
-		(at 121.92 185.42 0)
+		(at 116.84 185.42 0)
 		(unit 1)
 		(body_style 1)
@@
 		(fields_autoplaced yes)
 		(property "Reference" "TP4"
-			(at 124.46 180.8479 0)
+			(at 119.38 180.8479 0)
 			(show_name no)
 			(do_not_autoplace no)
@@
 		)
 		(property "Value" "GND"
-			(at 124.46 183.3879 0)
+			(at 119.38 183.3879 0)
 			(show_name no)
 			(do_not_autoplace no)
@@
 		)
 		(property "Footprint" "Connector_PinHeader_2.54mm:PinHeader_1x01_P2.54mm_Vertical"
-			(at 127 185.42 0)
+			(at 121.92 185.42 0)
 			(hide yes)
 			(show_name no)
@@
 		)
 		(property "Datasheet" ""
-			(at 127 185.42 0)
+			(at 121.92 185.42 0)
 			(hide yes)
 			(show_name no)
@@
 		)
 		(property "Description" "test point"
-			(at 121.92 185.42 0)
+			(at 116.84 185.42 0)
 			(hide yes)
 			(show_name no)
@@
 					(unit 1)
 				)
+			)
+		)
+	)
+	(symbol
+		(lib_id "Connector:TestPoint")
+		(at 125.73 185.42 0)
+		(unit 1)
+		(body_style 1)
+		(exclude_from_sim no)
+		(in_bom yes)
+		(on_board yes)
+		(in_pos_files yes)
+		(dnp no)
+		(fields_autoplaced yes)
+		(property "Reference" "TP10"
+			(at 128.27 180.8479 0)
+			(show_name no)
+			(do_not_autoplace no)
+			(effects
+				(font
+					(size 1.27 1.27)
+				)
+				(justify left)
+			)
+		)
+		(property "Value" "GND"
+			(at 128.27 183.3879 0)
+			(show_name no)
+			(do_not_autoplace no)
+			(effects
+				(font
+					(size 1.27 1.27)
+				)
+				(justify left)
+			)
+		)
+		(property "Footprint" "Connector_PinHeader_2.54mm:PinHeader_1x01_P2.54mm_Vertical"
+			(at 130.81 185.42 0)
+			(hide yes)
+			(show_name no)
+			(do_not_autoplace no)
+			(effects
+				(font
+					(size 1.27 1.27)
+				)
+			)
+		)
+		(property "Datasheet" ""
+			(at 130.81 185.42 0)
+			(hide yes)
+			(show_name no)
+			(do_not_autoplace no)
+			(effects
+				(font
+					(size 1.27 1.27)
+				)
+			)
+		)
+		(property "Description" "test point"
+			(at 125.73 185.42 0)
+			(hide yes)
+			(show_name no)
+			(do_not_autoplace no)
+			(effects
+				(font
+					(size 1.27 1.27)
+				)
+			)
+		)
+		(pin "1"
+		)
+		(instances
+			(project "Rainworks_Electrical"
+				(path "/86a7b6ea-a387-471e-a4e6-e2389d5f82ef"
+					(reference "TP10")
+					(unit 1)
+				)
